Commit message: add state graph

File: src/common/nhk2025b_description/urdf/nhk2025b.urdf (robot description, URDF)
Before this commit: robot nhk2025b, 13 links, 12 joints
Joints:
- joint l_pylon_arm_height_to_l_pylon_arm: origin xyz=0 0 0 rpy=0.0 0.0 0.0 -> xyz=0 0 0 rpy=0.0 1.5707963267948966 0.0
- joint r_pylon_arm_height_to_r_pylon_arm: origin xyz=0 0 0 rpy=0.0 0.0 0.0 -> xyz=0 0 0 rpy=0.0 1.5707963267948966 0.0
